File: Adapter-IO4-LED.brd (EAGLE design)
At the start: 30.9 x 31.9 mm, 7 parts

Commit message: added values for connectors
Parts:
- J1: value (none) -> RJ12/6
- JP1, JP2, JP3, JP4: value (none) -> 0.100
- RN1: value (none) -> 1K0
Changed lines of the file:
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@@
 <elements>
 <element name="U$1" library="SPCoast" package="OSHW-LOGO-M" value="DOC-OSHW-LOGO-M" x="26.67" y="27.94"/>
-<element name="J1" library="SPCoast" package="RJ25-PANEL" value="" x="15.24" y="26.67" smashed="yes" rot="R180">
+<element name="J1" library="SPCoast" package="RJ25-PANEL" value="RJ12/6" x="15.24" y="26.67" smashed="yes" rot="R180">
 <attribute name="NAME" x="13.335" y="29.21" size="1.778" layer="25"/>
 <attribute name="VALUE" x="22.225" y="34.29" size="1.778" layer="27" rot="R180"/>
@@
 <attribute name="OPL" value="none" x="15.24" y="26.67" size="1.778" layer="27" rot="R180" display="off"/>
 </element>
-<element name="JP1" library="SPCoast" package="1X02_LOCK" value="" x="16.51" y="5.08" rot="R90"/>
-<element name="JP2" library="SPCoast" package="1X02_LOCK" value="" x="13.97" y="5.08" rot="R90"/>
-<element name="JP3" library="SPCoast" package="1X02_LOCK" value="" x="11.43" y="5.08" rot="R90"/>
-<element name="JP4" library="SPCoast" package="1X02_LOCK" value="" x="8.89" y="5.08" rot="R90"/>
-<element name="RN1" library="resistor-sil" package="SIL5" value="" x="2.54" y="7.62" rot="R270">
+<element name="JP1" library="SPCoast" package="1X02_LOCK" value="0.100" x="16.51" y="5.08" rot="R90"/>
+<element name="JP2" library="SPCoast" package="1X02_LOCK" value="0.100" x="13.97" y="5.08" rot="R90"/>
+<element name="JP3" library="SPCoast" package="1X02_LOCK" value="0.100" x="11.43" y="5.08" rot="R90"/>
+<element name="JP4" library="SPCoast" package="1X02_LOCK" value="0.100" x="8.89" y="5.08" rot="R90"/>
+<element name="RN1" library="resistor-sil" package="SIL5" value="1K0" x="2.54" y="7.62" rot="R270">
 <attribute name="MF" value="" x="2.54" y="7.62" size="1.778" layer="27" rot="R270" display="off"/>
 <attribute name="MPN" value="" x="2.54" y="7.62" size="1.778" layer="27" rot="R270" display="off"/>

Commit message: normalized values
Parts:
- U$1: value DOC-OSHW-LOGO-M -> OSHW
Changed lines of the file:
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@@
 </autorouter>
 <elements>
-<element name="U$1" library="SPCoast" package="OSHW-LOGO-M" value="DOC-OSHW-LOGO-M" x="26.67" y="27.94"/>
+<element name="U$1" library="SPCoast" package="OSHW-LOGO-M" value="OSHW" x="26.67" y="27.94"/>
 <element name="J1" library="SPCoast" package="RJ25-PANEL" value="RJ12/6" x="15.24" y="26.67" smashed="yes" rot="R180">
 <attribute name="NAME" x="13.335" y="29.21" size="1.778" layer="25"/>
